File: src/pr-mini-bot.kicad_pcb (KiCad board)
At the start: 2 copper layers, 90 x 80 mm, 30 parts

Commit message: finish pcb
Parts:
- moved H8 1.00 mm to (246.0, 109.0)
Routing:
- net GND: vias 348 -> 284
Other:
- outline, holes or cut-outs redrawn
- board text added: "0 in"
- board text added: "0cm"
- board text added: "1"
- board text added: "2"
- board text added: "2 in"
- board text added: "3"
- board text added: "4"
- board text added: "5cm"
- board text added: "Ella-Rae Howells Malikai Bradford Damon Belohorec Ronan Dafoe Alex Brodie Claire Mannings Hung Pham Logan Petet"
- board text added: "Felix Atienza - Team Lead tobycm - Lead Coder Jordan Green - Build Team Lead Taylor Gordon - Electrical Lead"
- board text added: "Honourable mentions: Parents and sponsors"
- board text added: "Mentors: Joshua Walker Dave Hylands Marcus Francisco Dave Brodie"
- board text added: "Penticton Robotics 2025 TallyNuff Mini bot"
- board text added: "Scarlett Steyn Mason Price Zen Ritcey Keaton Sidorchuk Daphne LeBlanc Gurshan Bajwa"
- board text added: "Thank you to everyone for making the 2025 season a big success!!"
- board text added: "Until next time!! pentictonrobotics.ca"
- board text added: "made by tobycm https://tobycm.dev"
